File: E80-1800-pcb-universal/E80-1800-Matrix.kicad_sch (KiCad schematic)
At the start: 397 parts

Commit message: add 2x 1u to np_ent and add 2u np_+
Parts:
- added D173, D174, D175: 3mm, marbastlib-mx:LED_MX_3mm, symbol Device:LED_Small
- added R122: 560, Resistor_SMD:R_0603_1608Metric, symbol Device:R_Small
- added S8: (no value), symbol marbastlib-mx:MX_stab
- added SW3, SW4, SW5: (no value), symbol marbastlib-mx:MX_SW_solder
Connections:
- net +5V: now also D173.2 (A), D174.2 (A), D175.2 (A)
- net COL18: now also SW3.1, SW4.1, SW5.1
- net LED-: now also R122.1
- net at D33.1 (A), MX57.2: now also SW5.2
- net at D51.1 (A), MX96.2: now also SW3.2
- net at D115.1 (K), R71.2: now also D175.1 (K)
- net at D58.1 (A): now also SW4.2
- net at D154.1 (K), R107.2: now also D173.1 (K)
- new net: D174.1 (K), R122.2
- no-connect marks 2 -> 1

Commit message: add 2u 0 on numpad and rotary encoder
Parts:
- added D176: 3mm, marbastlib-mx:LED_MX_3mm, symbol Device:LED_Small
- added MX116: MX_SW_solder, marbastlib-mx:SW_MX_1u, symbol marbastlib-mx:MX_SW_solder
- added S9: (no value), symbol marbastlib-mx:MX_stab
- added SW6: (no value), symbol Device:RotaryEncoder_Switch
- S8: value (none) -> np_+; footprint (none) -> marbastlib-mx:STAB_MX_2u
- SW3, SW4, SW5: value (none) -> MX_SW_solder; footprint (none) -> marbastlib-mx:SW_MX_1u
Connections:
- net +5V: now also D176.2 (A)
- net COL16: now also MX116.1
- net COL18: now also SW6.S2
- net at D13.1 (A), MX17.2: now also SW6.S1
- net at D57.1 (A), MX114.2: now also MX116.2
- net at D171.1 (K), R120.2: now also D176.1 (K)
- new net GND: SW6.C
- new net SPI_MISO: SW6.B
- new net SPI_MOSI: SW6.A
