File: E80-1800-pcb-universal/E80-1800-Matrix.kicad_sch (KiCad schematic)
At the start: 409 parts, among them SW3 MX_SW_solder, SW4 MX_SW_solder, SW5 MX_SW_solder, SW6 RotaryEncoder_Switch

Commit message: prepare for jlcpcb
Connections:
- net SPI_MISO renamed ENCB
- net SPI_MOSI renamed ENCA
Changed lines of the file:
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@@
+    )
+  )
+  (global_label "ENCA" (shape input) (at 438.912 62.23 0) (fields_autoplaced)
+    (effects (font (size 1.27 1.27)) (justify left))
+    (property "Intersheet References" "${INTERSHEET_REFS}" (id 0) (at 446.0743 62.1506 0)
+      (effects (font (size 1.27 1.27)) (justify left) hide)
     )
   )
@@
     )
   )
+  (global_label "ENCB" (shape input) (at 438.912 57.15 0) (fields_autoplaced)
+    (effects (font (size 1.27 1.27)) (justify left))
+    (property "Intersheet References" "${INTERSHEET_REFS}" (id 0) (at 446.2557 57.0706 0)
+      (effects (font (size 1.27 1.27)) (justify left) hide)
+    )
+  )
   (global_label "COL09" (shape input) (at 222.25 50.8 90) (fields_autoplaced)
     (effects (font (size 1.27 1.27)) (justify left))
@@
     (property "Intersheet References" "${INTERSHEET_REFS}" (id 0) (at -29.21 12.7 0)
       (effects (font (size 1.27 1.27)) hide)
-    )
-  )
-  (global_label "SPI_MISO" (shape input) (at 438.912 57.15 0) (fields_autoplaced)
-    (effects (font (size 1.27 1.27)) (justify left))
-    (property "Intersheet References" "${INTERSHEET_REFS}" (id 0) (at 449.8843 57.0706 0)
-      (effects (font (size 1.27 1.27)) (justify left) hide)
     )
   )
@@
       (effects (font (size 1.27 1.27)) hide)
     )
-  )
-  (global_label "SPI_MOSI" (shape input) (at 438.912 62.23 0) (fields_autoplaced)
-    (effects (font (size 1.27 1.27)) (justify left))
-    (property "Intersheet References" "${INTERSHEET_REFS}" (id 0) (at 334.772 38.1 0)
-      (effects (font (size 1.27 1.27)) hide)
-    )
